Commit message: change package name

File: urdf/robotcraft2019.urdf (robot description, URDF)
Before this commit: robot robotcraft2019, 8 links, 7 joints
Links:
- link acrylic_base: geometry visual mesh filename=package://robotcraft-model-description/mesh/Transparent.stl scale=0.001 0.001 0.001
- link arduino: geometry visual mesh filename=package://robotcraft-model-description/mesh/Green.stl scale=0.001 0.001 0.001
- link base_link: geometry visual mesh filename=package://robotcraft-model-description/mesh/Black.stl scale=0.001 0.001 0.001
- link battery: geometry visual mesh filename=package://robotcraft-model-description/mesh/Purple.stl scale=0.001 0.001 0.001
- link bottom_base: geometry visual mesh filename=package://robotcraft-model-description/mesh/White.stl scale=0.001 0.001 0.001
